File: solanum-v2.kicad_sch (KiCad schematic)
At the start: 28 parts, among them J1 Battery_Cell, J2 AudioJack4, SW1 SW_Push_45deg, SW10 SW_Push_45deg, SW11 SW_Push_45deg, SW12 SW_Push_45deg, SW13 SW_Push_45deg, SW14 SW_Push_45deg, SW15 SW_Push_45deg, SW16 SW_Push_45deg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

Commit message: progress on v2 pcb
Parts:
- J1: footprint Library:JST_PH_S2B-PH-K_1x02_P2.00mm_Horizontal -> Connector_JST:JST_PH_S2B-PH-K_1x02_P2.00mm_Horizontal
Connections:
- net RAW: now also SW18.3 (C); no longer SW18.2 (B)
- net at J1.2 (Pin_2): now also SW18.2 (B); no longer SW18.3 (C)
Other:
- moved on the sheet: SW18

Commit message: fine tuning
Parts:
- SW18: footprint Library:SW_Slide_SPDT_Angled_CK_OS102011MA1Q -> Button_Switch_SMD:SW_SPDT_Shouhan_MSK12C02
Changed lines of the file:
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@@
 			)
 		)
-		(property "Footprint" "Library:SW_Slide_SPDT_Angled_CK_OS102011MA1Q"
+		(property "Footprint" "Button_Switch_SMD:SW_SPDT_Shouhan_MSK12C02"
 			(at 140.97 49.53 0)
 			(effects
